File: Beach40_kicad/beach40_kicad.kicad_pcb (KiCad board)
At the start: 2 copper layers, 200 x 100 mm, 81 parts, among them K1 RELAY_2RT, P1 LO In, P2 MIC_IN, P3 Audio Out, P4 ANT, Q1 BC548, Q2 2N2222, Q3 BD139, Q4 BD139, Q5 BC548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

Commit message: couple more tracks!
Parts:
- moved PTT1 128.7 mm to (182.0, 85.0)
- moved R15 48.7 mm to (181.0, 112.0)
- moved C9 35.4 mm to (189.0, 101.6)
- moved L7 33.6 mm to (180.0, 104.0), turned to 270 degrees
- moved C32 26.4 mm to (185.9, 68.1), turned to 0 degrees
- moved C10 26.2 mm to (193.3, 63.0)
- moved C26 19.0 mm to (191.0, 90.0)
Routing:
- net T/R-P-NO: track 193.9 -> 301.8 mm
- net Net-(K1-Pad8): track 0.00 -> 24.8 mm
- net T/R-P-NC: track 0.40 -> 21.6 mm
- net +12V: track 0.00 -> 8.84 mm
- net Net-(K1-Pad9): track 0.00 -> 6.81 mm
- net Net-(L2-Pad1): track 41.9 -> 48.3 mm
- net Net-(C10-Pad1): track 0.00 -> 5.16 mm
