File: Beach40_kicad/beach40_kicad.kicad_pcb (KiCad board)
At the start: 2 copper layers, 200 x 100 mm, 81 parts, among them K1 RELAY_2RT, P1 LO In, P2 MIC_IN, P3 Audio Out, P4 ANT, Q1 BC548, Q2 2N2222, Q3 BD139, Q4 BD139, Q5 BC548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

Commit message: more mucking about!
Parts:
- moved L9 53.8 mm to (201.0, 83.7)

Commit message: mucking about more with layout, a bit thinner!
Parts:
- moved Q4 71.6 mm to (160.9, 75.8)
- moved Q3 55.1 mm to (203.2, 93.9)
- moved L2 53.3 mm to (193.9, 79.9), turned to 0 degrees
- moved C20 52.2 mm to (182.1, 91.8), turned to 270 degrees
- moved R15 51.8 mm to (170.4, 93.7), turned to 0 degrees
- moved C23 48.9 mm to (165.9, 97.7), turned to 180 degrees
- moved C21 47.7 mm to (181.7, 94.0), turned to 270 degrees
- moved R17 42.4 mm to (173.1, 97.7), turned to 180 degrees
- moved R14 40.4 mm to (182.4, 97.8), turned to 270 degrees
- moved R16 36.6 mm to (173.0, 100.9), turned to 180 degrees
- moved K1 32.1 mm to (137.4, 98.6), turned to 0 degrees
- moved L9 20.8 mm to (221.8, 83.8)
- moved C25 19.7 mm to (156.7, 85.7)
- moved R18 16.3 mm to (152.8, 83.0)
- moved C29 16.3 mm to (152.9, 76.8)
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Routing:
- net Net-(C20-Pad1): track 101.6 -> 0.00 mm, vias 1 -> 0
- net T/R-S-NC: track 57.7 -> 0.00 mm
- net LPF: track 61.8 -> 7.30 mm
- net Net-(C29-Pad2): track 63.4 -> 10.1 mm
- net T/R-P-NO: track 199.0 -> 154.1 mm, vias 3 -> 2
- net Net-(C25-Pad1): track 53.2 -> 8.71 mm
- net Net-(L2-Pad1): track 47.0 -> 5.10 mm
- net T/R-S-NO: track 6.54 -> 0.00 mm
- net Net-(C25-Pad2): track 5.67 -> 0.00 mm
