File: my_LBS/My_LBS.sch (KiCad schematic (older format))
At the start: 13 parts

Commit message: updates updates updates!
Parts:
- removed C? (x5): 100n, symbol C
- removed L?: Bifilar_10t_choke, symbol Bifilar_10t_choke
- removed Q?: 2n3904, symbol NPN
- removed R?: 470, symbol R
- removed R?: 1k, symbol R
- removed R?: 330, symbol R
- removed R?: 4.7, symbol R
- removed R?: 15, symbol R
- removed RV?: 100, symbol POT
- added C1, C2, C3, C4, C5, C6: 100n, symbol C
- added C10, C12, C15: 220u, FT:CAP_ELECTRO_D4S1.8, symbol C_POL
- added C11: 47u, FT:CAP_ELECTRO_D4S1.8, symbol C_POL
- added C13: 4.7n, FT:1210_CAP, symbol CAP
- added C14: 100n, FT:1210_CAP, symbol CAP
- added C7, C8: 4.7u, symbol CP1
- added C9: 4.7u, FT:CAP_ELECTRO_D4S1.8, symbol C_POL
- added C? (x2): 53.2p, symbol CAP_TRIM
- added C?: 7.2p, symbol CAP_TRIM
- added C? (x2): 181.6p, symbol CAP_TRIM
- added L1: Bifilar_10t_choke, symbol Bifilar_10t_choke
- added L? (x2): INDUCTOR, symbol INDUCTOR
- added P1: Audio Out, Pin_Headers:Pin_Header_Straight_1x02, symbol CONN_01X02
- added P? (x2): BNC, symbol BNC
- added Q1, Q2: 2n3904, symbol NPN
- added R1: 470, symbol R
- added R10: 2.2k, FT:1210, symbol R
- added R11: 2.2, FT:1210, symbol R
- added R2: 1k, symbol R
- added R3: 330, symbol R
- added R4: 4.7, symbol R
- added R5: 15, symbol R
- added R6: 10k, symbol R
- added R7: 100k, symbol R
- added R8: 10, FT:1210, symbol R
- added R9: 18, FT:1210, symbol R
- added RV1: 100, symbol POT
- added RV2: 10k, symbol POT
- added U1: ADE-1, symbol ADE-1
- added U2: LM386, Housings_SOIC:SOIC-8-1EP_3.9x4.9mm_Pitch1.27mm, symbol LM386
Connections:
- net labels added: +12VR, AUDIO, FILTER, T/R-P-NC
- net labels removed: CLK_IN
- wire segments 20 -> 90
- no-connect marks 0 -> 1
Other:
- note added: "20 Turns bifilar t-86-6"

Commit message: Corrected 10t bifilar choke. updates to LBS making it as built, and to re-fit the 10t choke.
Parts:
- removed C9: 4.7u, FT:CAP_ELECTRO_D4S1.8, symbol C_POL
- added C16: 10u, symbol C_POL
- added C17: 100u, symbol C_POL
- added C18: 100n, symbol C
- added C9: 100n, symbol CAP
- added D1: DIODE, symbol DIODE
- added R12: 10, symbol R
- added R13: 470 1/2W, symbol R
- gave numbers to parts that had none: 9
Connections:
- net labels removed: +12VR
- wire segments 90 -> 102
- no-connect marks 1 -> 0
Other:
- moved on the sheet: C4, C5, C8, L1, R5

Commit message: fixed conflicts for Beach40
Parts:
- removed C12: 220u, FT:CAP_ELECTRO_D4S1.8, symbol C_POL
- C13: renamed from C10; value 220u -> 100u
- renumbered C4 to C10, C5 to C11, C8 to C12, C11 to C14, C13 to C16, C14 to C17, C15 to C18, C6 to C2, C2 to C3, C7 to C4, C9 to C5, C3 to C6, C16 to C7, C17 to C8, C18 to C9, P2 to P1, P1 to P2, R8 to R10, R9 to R11, R10 to R12, R11 to R13, R6 to R5, R7 to R6, R12 to R7, R13 to R8, R5 to R9
Connections:
- wire segments 102 -> 100
Other:
- moved on the sheet: C2, C4, C5, C7, C8, C9, Q2, R5, R6, R7, R8, RV1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
